File: pic18/pic18.kicad_pcb (KiCad board)
At the start: 2 copper layers, 90.2 x 99.1 mm, 82 parts, among them J1 PORTA, J10 PORTD, J11 PORTD1, J12 PORTC, J13 PORTC1, J14 PICKIT3, J15 CONTROL, J16 5V, J17 3.3V, J18 5V, J19 3.3V, J2 PORTB, J20 LED'S, J21 BUZZER, J22 PORTE, J23 PORTE1, J3 USB_B, J4 Barrel_Jack_Switch, J5 TECLADO, J6 LCD, J7 PORTA1, J8 HC-05, J9 PORTB1, Q1 2N3906, SW1 SW_Push, SW2 SW_DIP_x01, U1 PIC18F45K50, U3 NRF24L01_Breakout

Commit message: javimenba
Parts:
- J3: value USB_B -> USB_B_Micro; footprint Connector_USB:USB_B_OST_USB-B1HSxx_Horizontal -> Connector_USB:USB_Micro-B_Wuerth_629105150521; moved to B.Cu
- J6: value LCD -> Conn_01x04; footprint Connector_PinSocket_2.54mm:PinSocket_1x16_P2.54mm_Vertical -> Connector_PinSocket_2.54mm:PinSocket_1x04_P2.54mm_Vertical
- moved J6 16.3 mm to (185.4, 91.4)
- moved J3 12.7 mm to (120.7, 137.2), turned to 180 degrees
- moved R1 7.00 mm to (120.5, 129.5)
Connections:
- J3 pad 2: /RC4 -> Net-(J3-Pad2)
- J3 pad 4: GND -> Net-(J3-Pad4)
- J6 pad 3: Net-(J6-Pad3) -> /RB1
- J6 pad 4: /RD1 -> /RB0
- R19 pad 1: Net-(R19-Pad1) -> Net-(C8-Pad1)
- R8 pad 2: Net-(R19-Pad1) -> Net-(C8-Pad1)
- SW1 pad 1: Net-(C8-Pad1) -> GND
- SW1 pad 2: Net-(R19-Pad1) -> Net-(C8-Pad1)
Routing:
- net GND: track 444.7 -> 0.00 mm
- net /GND1: track 45.6 -> 106.2 mm
- net /RB1: track 150.8 -> 208.7 mm, vias 1 -> 0
- net /RD1: track 125.8 -> 71.4 mm
- net /RD2: track 124.7 -> 74.4 mm, vias 1 -> 0
- net /RC2: track 66.7 -> 116.2 mm
- net /RD3: track 120.6 -> 71.3 mm
- net /RB0: track 158.6 -> 198.6 mm, vias 1 -> 0
- net /RC4: track 39.1 -> 0.00 mm
- net /RD6: track 89.0 -> 50.8 mm
- net /RD7: track 85.8 -> 47.7 mm
- net /RD5: track 91.0 -> 53.4 mm
- net /RD4: track 93.7 -> 57.0 mm
- net Net-(BZ1-Pad1): track 33.3 -> 69.0 mm
- net Net-(J6-Pad15): track 21.1 -> 0.00 mm
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Other:
- net class Default added: clearance 0.254, trace_width 0.254, via_dia 0.762, via_drill 0.381
- board text added: "OLED"
- board text added: "VERSION 2.0"
- board text removed: "LCD"
- board text removed: "VERSION 1.0"

Commit message: JaPic
Parts:
- removed G: LOGO, FIMEE:abeja
- removed J3: USB_B_Micro, Connector_USB:USB_Micro-B_Wuerth_629105150521
- removed JAPIC: LOGO, FIMEE:japic
- added G***: LOGO, FIMEE:japic, B.Cu at (173.6, 82.4)
- added G***: LOGO, FIMEE:usb_logo, F.Cu at (156.3, 135.1)
- added G***: LOGO, FIMEE:abeja_sf, F.Cu at (106.7, 61.0)
- added G***: LOGO, FIMEE:open_hardware, B.Cu at (101.5, 65.7)
- added G***: LOGO, FIMEE:kicad_logo, B.Cu at (101.2, 57.2)
- added INT0: SW_Push, Button_Switch_SMD:SW_SPST_CK_RS282G05A3, F.Cu at (157.5, 59.7)
- added INT1: SW_Push, Button_Switch_SMD:SW_SPST_CK_RS282G05A3, F.Cu at (165.1, 59.7)
- added INT2: SW_Push, Button_Switch_SMD:SW_SPST_CK_RS282G05A3, F.Cu at (172.7, 59.7)
- added Q2: 2N2219, Package_TO_SOT_THT:TO-92_Inline, F.Cu at (146.1, 137.2)
- added Q3: 2N2219, Package_TO_SOT_THT:TO-92_Inline, F.Cu at (146.1, 124.5)
- added Q4: 2N2219, Package_TO_SOT_THT:TO-92_Inline, F.Cu at (146.1, 130.8)
- added R23: 10k, Resistor_SMD:R_1206_3216Metric, B.Cu at (176.5, 59.7)
- added R24: 10K, Resistor_SMD:R_1206_3216Metric, F.Cu at (139.7, 138.4)
- added R25: 1K, Resistor_SMD:R_1206_3216Metric, B.Cu at (114.3, 132.1)
- added R26: 1K, Resistor_SMD:R_1206_3216Metric, B.Cu at (113.7, 124.7)
- added R27: 1K, Resistor_SMD:R_1206_3216Metric, B.Cu at (118.5, 132.1)
- added R28: 1K, Resistor_SMD:R_1206_3216Metric, B.Cu at (125.7, 124.5)
- added R29: 1K, Resistor_SMD:R_1206_3216Metric, B.Cu at (133.1, 132.1)
- added R30: 1K, Resistor_SMD:R_1206_3216Metric, B.Cu at (119.4, 124.5)
- added R31: 1K, Resistor_SMD:R_1206_3216Metric, B.Cu at (125.9, 132.1)
- added R32: 1K, Resistor_SMD:R_1206_3216Metric, B.Cu at (132.1, 124.5)
- added R33: 10K, Resistor_SMD:R_1206_3216Metric, F.Cu at (139.7, 132.1)
- added R37: 10K, Resistor_SMD:R_1206_3216Metric, F.Cu at (139.7, 125.7)
- added U2: 3x7Segment, Javi-7SegDisplays:3x7SEGMENT-04x08-Red, F.Cu at (125.7, 132.1)
- added USB1: HRO-TYPE-C-31-M-12, TypeC:HRO-TYPE-C-31-M-12-HandSoldering, B.Cu at (156.2, 141.0)
- C4: footprint Capacitor_THT:CP_Radial_D10.0mm_P2.50mm -> Capacitor_THT:CP_Radial_D5.0mm_P2.50mm
- R1: value 10K -> 5.1k
- R10: value 220 -> 5.1k
- R20: value 220 -> 10k
- R21: value 1k -> 10k
- moved J5 59.4 mm to (185.4, 70.1), turned to 0 degrees
- moved R10 52.2 mm to (158.9, 127.0), turned to 270 degrees
- moved R20 47.9 mm to (160.0, 59.7), turned to 270 degrees
- moved 3.3v1 47.3 mm to (177.8, 111.8), turned to 90 degrees
- moved R5 46.1 mm to (165.1, 104.0), turned to 90 degrees
- moved C4 43.4 mm to (158.8, 82.5)
- moved R21 41.0 mm to (167.6, 59.7), turned to 90 degrees
- moved C7 40.7 mm to (169.0, 114.3), turned to 180 degrees
- moved R4 39.5 mm to (172.7, 104.1), turned to 270 degrees
- moved J4 35.3 mm to (174.0, 121.9), turned to 180 degrees
- moved R1 33.2 mm to (153.7, 127.0), turned to 90 degrees
- moved R8 31.4 mm to (133.3, 66.0)
- moved RV1 29.2 mm to (158.8, 72.4)
- moved R19 26.8 mm to (133.3, 60.8)
- moved C6 26.7 mm to (158.8, 91.4)
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Connections:
- R1 pad 2: /VUSB -> Net-(R1-Pad2)
- R10 pad 1: VDD -> GND
- R20 pad 1: Net-(J6-Pad3) -> /RB0
- R21 pad 1: VDD -> /RB1
- R21 pad 2: Net-(J6-Pad3) -> GND
Routing:
- net /RB1: track 208.7 -> 0.00 mm
- net VDD: track 208.6 -> 0.00 mm
- net /RB0: track 198.6 -> 0.00 mm
- net /RB7: track 178.4 -> 0.00 mm
- net /RB5: track 174.8 -> 0.00 mm
- net /RB6: track 167.5 -> 0.00 mm, vias 1 -> 0
- net /RB2: track 161.6 -> 0.00 mm, vias 1 -> 0
- net /RB4: track 147.4 -> 0.00 mm
- net /RB3: track 146.5 -> 0.00 mm, vias 1 -> 0
- net 3.3v: track 136.9 -> 0.00 mm
- net /RC2: track 116.2 -> 0.00 mm
- net /MCLR: track 115.8 -> 0.00 mm, vias 2 -> 0
- net /GND1: track 106.2 -> 0.00 mm
- net /RE0: track 102.0 -> 0.00 mm
- net /RE1: track 95.9 -> 0.00 mm, vias 1 -> 0
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- removed copper zone on B.Cu, net GND
- removed copper zone on F.Cu, net GND
Other:
- board text added: "2.5"
- board text removed: "1"
- board text removed: "16"
- board text removed: "VERSION 2.0"

Commit message: JaPic
Parts:
- removed 3.3v1, 5v1: L7805, Package_TO_SOT_THT:TO-220-3_Vertical
- removed C6: 0.33uf, Capacitor_THT:CP_Radial_D5.0mm_P2.50mm
- removed C7: 100nf, Capacitor_SMD:C_1206_3216Metric
- removed D2: 1N4148, Diode_THT:D_DO-35_SOD27_P7.62mm_Horizontal
- removed D3: LED, LED_SMD:LED_0805_2012Metric
- removed the G*** at (173.6, 82.4)
- removed the G*** at (106.7, 61.0)
- removed the G*** at (101.5, 65.7)
- removed the G*** at (101.2, 57.2)
- removed the G*** at (171.4, 85.1)
- removed H4: MountingHole, MountingHole:MountingHole_4mm_Pad_Via
- removed J13: PORTC1, Connector_PinSocket_2.54mm:PinSocket_1x03_P2.54mm_Vertical
- removed J16, J18: 5V, Connector_PinSocket_2.54mm:PinSocket_1x02_P2.54mm_Vertical
- removed J17, J19: 3.3V, Connector_PinSocket_2.54mm:PinSocket_1x02_P2.54mm_Vertical
- removed J22: PORTE, Connector_PinSocket_2.54mm:PinSocket_1x03_P2.54mm_Vertical
- removed J23: PORTE1, Connector_PinSocket_2.54mm:PinSocket_1x03_P2.54mm_Vertical
- removed Q1: 2N3906, Package_TO_SOT_THT:TO-92_Inline
- removed Q2, Q3, Q4: 2N2219, Package_TO_SOT_THT:TO-92_Inline
- added C9: 0.1uF, Capacitor_SMD:C_0805_2012Metric, B.Cu at (76.5, 97.2)
- added D14: 1N4007, Diode_SMD:D_1210_3225Metric_Pad1.42x2.65mm_HandSolder, B.Cu at (71.5, 97.2)
- added DIG1: 2N2219, Package_TO_SOT_THT:TO-92_Inline, F.Cu at (93.6, 81.8)
- added DIG2: 2N2219, Package_TO_SOT_THT:TO-92_Inline, F.Cu at (93.6, 75.5)
- added DIG3: 2N2219, Package_TO_SOT_THT:TO-92_Inline, F.Cu at (93.6, 69.2)
- added G1: LOGO, FIMEE:japic, B.Cu at (89.8, 41.7)
- added G2: LOGO, FIMEE:kicad_logo, B.Cu at (99.8, 34.5)
- added G3: LOGO, FIMEE:open_hardware, B.Cu at (99.3, 41.9)
- added G4: LOGO, FIMEE:github, B.Cu at (98.8, 48.8)
- added G5: LOGO, FIMEE:fimee, F.Cu at (87.7, 60.8)
- added G6: LOGO, FIMEE:abeja_sf, F.Cu at (91.2, 37.8)
- added J3: Barrel_Jack_Switch, Connector_BarrelJack:BarrelJack_Wuerth_6941xx301002, F.Cu at (71.3, 86.0)
- added R34: 470, Resistor_SMD:R_0805_2012Metric, B.Cu at (54.6, 85.9)
- added U4: AMS1117-5.0, Package_TO_SOT_SMD:SOT-223-3_TabPin2, F.Cu at (83.2, 91.2)
- added U5: AMS1117-3.3, Package_TO_SOT_SMD:SOT-223-3_TabPin2, F.Cu at (91.4, 91.0)
- C3: value 100nf -> 100uF; footprint Capacitor_SMD:C_1206_3216Metric -> Capacitor_THT:CP_Radial_D5.0mm_P2.50mm; moved to F.Cu
- C4: value 220uf -> 0.1uF; footprint Capacitor_THT:CP_Radial_D5.0mm_P2.50mm -> Capacitor_SMD:C_0805_2012Metric; moved to B.Cu
- C5: value 100nf -> 0.1uF; footprint Capacitor_SMD:C_1206_3216Metric -> Capacitor_SMD:C_0805_2012Metric
- D1: value 1N4148 -> LED; footprint Diode_THT:D_DO-35_SOD27_P7.62mm_Horizontal -> LED_SMD:LED_0805_2012Metric
- D10: value LED -> LED10
- D11, D5: value LED -> LED11
- D4: value LED -> LED4
- D6: value LED -> LED6
- D7: value LED -> LED7
- D8: value LED -> LED8
- D9: value LED -> LED9
- H1: value MountingHole -> 1
- H2: value MountingHole -> 2
- H3: value MountingHole -> 3
- J1, J2: footprint Connector_PinSocket_2.54mm:PinSocket_1x08_P2.54mm_Vertical -> Connector_PinSocket_2.54mm:PinSocket_2x08_P2.54mm_Vertical
- J10: value PORTD -> PORTE; footprint Connector_PinSocket_2.54mm:PinSocket_1x08_P2.54mm_Vertical -> Connector_PinSocket_2.54mm:PinSocket_2x03_P2.54mm_Vertical
- J11: value PORTD1 -> 5v-3.3v; footprint Connector_PinSocket_2.54mm:PinSocket_1x08_P2.54mm_Vertical -> Connector_PinSocket_2.54mm:PinSocket_2x02_P2.54mm_Vertical
- J12: value PORTC -> 5v-3.3v; footprint Connector_PinSocket_2.54mm:PinSocket_1x03_P2.54mm_Vertical -> Connector_PinSocket_2.54mm:PinSocket_2x02_P2.54mm_Vertical
- J4: value Barrel_Jack_Switch -> Vin; footprint Connector_BarrelJack:BarrelJack_Horizontal -> Connector_PinHeader_2.54mm:PinHeader_1x02_P2.54mm_Vertical
- J6: value Conn_01x04 -> OLED
- J7: value PORTA1 -> PORTD; footprint Connector_PinSocket_2.54mm:PinSocket_1x08_P2.54mm_Vertical -> Connector_PinSocket_2.54mm:PinSocket_2x08_P2.54mm_Vertical
- J9: value PORTB1 -> PORTC; footprint Connector_PinSocket_2.54mm:PinSocket_1x08_P2.54mm_Vertical -> Connector_PinSocket_2.54mm:PinSocket_2x03_P2.54mm_Vertical
- R1, R10, R11, R12, R13, R14, R15, R16, R17, R18, R19, R20, R21, R22, R23, R25, R26, R27, R28, R29, R30, R31, R32, R6, R7, R8, R9: footprint Resistor_SMD:R_1206_3216Metric -> Resistor_SMD:R_0805_2012Metric
- R2, R3: value 5.6k -> 4.7; footprint Resistor_SMD:R_1206_3216Metric -> Resistor_SMD:R_0805_2012Metric
- R24, R33, R37: footprint Resistor_SMD:R_1206_3216Metric -> Resistor_SMD:R_0805_2012Metric; moved to B.Cu
- R4: value 10k -> 4.7; footprint Resistor_SMD:R_1206_3216Metric -> Resistor_SMD:R_0805_2012Metric
- R5: value 470 -> 4.7; footprint Resistor_SMD:R_1206_3216Metric -> Resistor_SMD:R_0805_2012Metric
- moved R2 141.2 mm to (56.6, 66.5), turned to 0 degrees
- moved H3 140.2 mm to (45.8, 95.4)
- moved R3 125.0 mm to (56.6, 64.0), turned to 0 degrees
- moved R4 123.7 mm to (56.6, 61.5), turned to 180 degrees
- moved SW1 122.8 mm to (38.8, 38.4), turned to 90 degrees
- moved D1 118.1 mm to (54.6, 83.7), turned to 0 degrees
- moved R5 117.5 mm to (56.6, 58.9), turned to 0 degrees
- moved R22 115.5 mm to (62.5, 85.9)
- moved H2 109.0 mm to (103.3, 24.4)
- moved R1 107.5 mm to (52.5, 90.6)
- moved USB1 105.8 mm to (58.7, 100.1)
- moved G*** 105.4 mm to (58.9, 94.7)
- moved R10 100.9 mm to (64.9, 90.6), turned to 90 degrees
- moved J11 98.5 mm to (46.1, 88.6), turned to 270 degrees
- moved D4 98.1 mm to (49.7, 48.7), turned to 0 degrees
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Connections:
- C1 pad 1: VDD -> Net-(C1-Pad1)
- C3 pad 1: Net-(5v1-Pad3) -> Net-(C3-Pad1)
- C4 pad 1: GND -> Net-(C3-Pad1)
- C4 pad 2: 5V -> GND
- C5 pad 1: VDD -> 3.3v
- D1 pad 1: GND -> Net-(D1-Pad1)
- D1 pad 2: Net-(5v1-Pad2) -> Net-(C3-Pad1)
- H1 pad 1: (no net) -> GND
- H2 pad 1: (no net) -> GND
- H3 pad 1: (no net) -> GND
- J1 pad 2: /RA1 -> /RA0
- J1 pad 3: /RA2 -> /RA1
- J1 pad 4: /RA3 -> /RA1
- J1 pad 5: /RA4 -> /RA2
- J1 pad 6: /RA5 -> /RA2
- J1 pad 7: /RA6 -> /RA3
- J1 pad 8: /RA7 -> /RA3
- J10 pad 1: /RD0 -> /RE0
- J10 pad 2: /RD1 -> /RE0
- J10 pad 3: /RD2 -> /RE1
- J10 pad 4: /RD3 -> /RE1
- J10 pad 5: /RD4 -> /RE2
- J10 pad 6: /RD5 -> /RE2
- J11 pad 1: /RD0 -> VDD
- J11 pad 2: /RD1 -> 3.3v
- J11 pad 3: /RD2 -> GND
- J11 pad 4: /RD3 -> GND
- J12 pad 1: /RC0 -> VDD
- J12 pad 2: /RC1 -> 3.3v
- J12 pad 3: /RC2 -> GND
- J2 pad 2: /RB1 -> /RB0
- J2 pad 3: /RB2 -> /RB1
- J2 pad 4: /RB3 -> /RB1
- J2 pad 5: /RB4 -> /RB2
- J2 pad 6: /RB5 -> /RB2
- J2 pad 7: /RB6 -> /RB3
- J2 pad 8: /RB7 -> /RB3
- J4 pad 1: Net-(5v1-Pad1) -> /Vin
- J7 pad 1: /RA0 -> /RD0
- J7 pad 2: /RA1 -> /RD0
- J7 pad 3: /RA2 -> /RD1
- J7 pad 4: /RA3 -> /RD1
- J7 pad 5: /RA4 -> /RD2
- J7 pad 6: /RA5 -> /RD2
- J7 pad 7: /RA6 -> /RD3
- J7 pad 8: /RA7 -> /RD3
- J9 pad 1: /RB0 -> /RC0
- J9 pad 2: /RB1 -> /RC0
- J9 pad 3: /RB2 -> /RC1
- J9 pad 4: /RB3 -> /RC1
- J9 pad 5: /RB4 -> /RC2
- J9 pad 6: /RB5 -> /RC2
- R2 pad 1: Net-(5v1-Pad3) -> VDD
- R2 pad 2: GND -> Net-(R2-Pad2)
- R25 pad 2: /RB6 -> /RD6
- R26 pad 2: /RB5 -> /RD5
- R27 pad 2: /RB4 -> /RD4
- R28 pad 2: /RB3 -> /RD3
- R29 pad 2: /RB2 -> /RD2
- R3 pad 1: Net-(Q1-Pad2) -> Net-(R2-Pad2)
- R3 pad 2: Net-(5v1-Pad3) -> Net-(R3-Pad2)
- R30 pad 2: /RB1 -> /RD1
- R31 pad 2: /RB0 -> /RD0
- R32 pad 2: /RB7 -> /RD7
- R4 pad 1: /VUSB -> Net-(R3-Pad2)
- R4 pad 2: GND -> Net-(R4-Pad2)
- R5 pad 1: Net-(D3-Pad2) -> Net-(R4-Pad2)
- R5 pad 2: 5V -> Net-(C1-Pad1)
- U1 pad 11: VDD -> Net-(C1-Pad1)
- U1 pad 32: VDD -> Net-(U1-Pad32)
- USB1 pad 11: /VUSB -> 5V
- USB1 pad 2: /VUSB -> 5V
Routing:
- net Net-(C3-Pad1): track 0.00 -> 28.5 mm, vias 0 -> 2
- net Net-(C9-Pad1): track 0.00 -> 20.3 mm, vias 0 -> 1
- net /Vin: track 0.00 -> 17.5 mm
- net GND: track 0.00 -> 1.62 mm
Other:
- board size 90.2 x 99.1 mm -> 71.1 x 80.4 mm
- board text added: "5v/USB/Vin"
- board text added: "@javimenba"
- board text added: "BUZER"
- board text added: "INT0"
- board text added: "INT1"
- board text added: "INT2"
- board text added: "LA0"
- board text added: "LA1"
- board text added: "LA2"
- board text added: "LA3"
- board text added: "LA4"
- board text added: "LA5"
- board text added: "LA6"
- board text added: "LA7"
- board text added: "MISQ"
- board text added: "PORTA"
- board text added: "PORTB"
- board text added: "PORTC"
- board text added: "PORTD"
- board text added: "PORTE"
- board text added: "Vin"
- board text removed: "2.5"
- board text removed: "5V/USB"
- board text removed: "ADC"
- board text removed: "BUZZER"
- board text removed: "MISO"
- board text removed: "OFF"
- board text removed: "ON"
- board text removed: "RA1"
- board text removed: "RA2"
- board text removed: "RA3"
- board text removed: "RA4"
- board text removed: "RA5"
- board text removed: "RA6"
- board text removed: "RB1"
- board text removed: "RB2"
- board text removed: "RB3"
- board text removed: "RB4"
- board text removed: "RB5"
- board text removed: "RB6"
- board text removed: "RC1"
- board text removed: "RD1"
- board text removed: "RD2"
- board text removed: "RD3"
- board text removed: "RD4"
- board text removed: "RD5"
- board text removed: "RD6"
- board text removed: "RE1"

Commit message: JaPic
Parts:
- moved J7 61.3 mm to (41.6, 63.5), turned to 0 degrees
- moved J2 61.2 mm to (88.8, 24.5), turned to 270 degrees
- moved J1 16.7 mm to (49.6, 21.9), turned to 90 degrees
- moved R1 13.5 mm to (65.1, 95.3)
Routing:
- net GND: track 1.62 -> 213.4 mm, vias 0 -> 2
- net /RB7: track 0.00 -> 69.2 mm
- net /RB2: track 0.00 -> 69.1 mm, vias 0 -> 1
- net /RB0: track 0.00 -> 68.2 mm
- net /RB1: track 0.00 -> 66.8 mm, vias 0 -> 2
- net /RB6: track 0.00 -> 65.6 mm
- net /RA6: track 0.00 -> 62.7 mm, vias 0 -> 1
- net /RB5: track 0.00 -> 61.6 mm, vias 0 -> 1
- net /RA7: track 0.00 -> 58.5 mm, vias 0 -> 1
- net /RB4: track 0.00 -> 58.1 mm, vias 0 -> 1
- net /RB3: track 0.00 -> 56.0 mm, vias 0 -> 2
- net VPICKIT3: track 0.00 -> 47.8 mm, vias 0 -> 1
- net 5V: track 0.00 -> 45.4 mm, vias 0 -> 1
- net /RA5: track 0.00 -> 37.6 mm
- net /RA4: track 0.00 -> 35.7 mm
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
Commit message: JaPic
Parts:
- moved R29 19.5 mm to (103.7, 82.1), turned to 180 degrees
- moved R26 19.3 mm to (98.3, 63.4)
- moved R25 2.82 mm to (99.4, 82.2)
- turned R6 to 270 degrees
- turned R7 to 270 degrees
Routing:
- net GND: track 213.4 -> 338.9 mm, vias 2 -> 6
- net /RD6: track 0.00 -> 115.8 mm, vias 0 -> 5
- net /RD7: track 0.00 -> 105.1 mm, vias 0 -> 4
- net /RD1: track 0.00 -> 104.4 mm, vias 0 -> 9
- net /RD3: track 0.00 -> 101.5 mm, vias 0 -> 3
- net /RD0: track 0.00 -> 86.3 mm, vias 0 -> 5
- net /RD5: track 0.00 -> 85.5 mm, vias 0 -> 2
- net /RD2: track 0.00 -> 79.5 mm, vias 0 -> 3
- net /RB7: track 69.2 -> 142.8 mm, vias 0 -> 5
- net /RB6: track 65.6 -> 134.9 mm, vias 0 -> 5
- net /RB5: track 61.6 -> 124.4 mm, vias 1 -> 5
- net /RE1: track 0.00 -> 57.6 mm, vias 0 -> 1
- net /RD4: track 0.00 -> 48.9 mm, vias 0 -> 1
- net VDD: track 0.00 -> 44.4 mm
- net Net-(BZ1-Pad1): track 0.00 -> 42.8 mm, vias 0 -> 3
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- added copper zone on B.Cu, net GND
- added copper zone on F.Cu, net GND

Commit message: JaPic
Parts:
- added H4: 4, MountingHole:MountingHole_4mm_Pad_Via, F.Cu at (103.0, 95.5)
Routing:
- net VDD: track 44.4 -> 237.8 mm, vias 0 -> 9
- net 3.3v: track 25.3 -> 170.9 mm, vias 1 -> 10
- net GND: track 338.9 -> 481.0 mm, vias 6 -> 14
- net (no net): track 0.00 -> 130.9 mm
- net /MCLR: track 13.3 -> 116.3 mm, vias 0 -> 4
- net /RD4: track 48.9 -> 117.8 mm, vias 1 -> 7
- net /RE2: track 22.8 -> 86.8 mm, vias 1 -> 6
- net /RE0: track 33.2 -> 92.8 mm, vias 1 -> 7
- net /RE1: track 57.6 -> 98.4 mm, vias 1 -> 6
- net Net-(C3-Pad1): track 30.3 -> 60.1 mm, vias 2 -> 6
- net /RB1: track 99.2 -> 120.7 mm, vias 5 -> 6
- net /RB7: track 142.8 -> 153.1 mm
- net /RB6: track 134.9 -> 141.2 mm
- net /RB5: track 124.4 -> 129.8 mm
- net Net-(R10-Pad2): track 10.6 -> 15.1 mm
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- removed copper zone on B.Cu, net GND
- removed copper zone on F.Cu, net GND

Commit message: JaPic
Parts:
- removed G1: LOGO, FIMEE:japic
- C5, C9, D14: moved to F.Cu
- moved G2 57.7 mm to (47.1, 58.0)
- moved G3 57.7 mm to (46.6, 65.3)
- moved G4 57.7 mm to (46.1, 72.3)
- moved INT2 54.5 mm to (48.5, 74.8)
- moved D11 52.6 mm to (71.8, 78.7), turned to 180 degrees
- moved R29 52.3 mm to (71.0, 41.3)
- moved DIG1 51.8 mm to (93.2, 30.1), turned to 270 degrees
- moved C8 51.5 mm to (45.3, 86.7)
- moved SW1 51.2 mm to (42.4, 89.4)
- moved J7 51.0 mm to (71.1, 21.8), turned to 90 degrees
- moved J21 50.6 mm to (95.6, 64.0), turned to 270 degrees
- moved R32 50.2 mm to (71.3, 36.7), turned to 180 degrees
- moved U1 49.6 mm to (67.8, 78.2), turned to 180 degrees
- moved R24 49.3 mm to (97.0, 31.6), turned to 90 degrees
- moved R31 49.3 mm to (71.5, 33.4), turned to 180 degrees
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Routing:
- net GND: track 481.0 -> 87.1 mm, vias 14 -> 3
- net VDD: track 237.8 -> 0.00 mm, vias 9 -> 0
- net 3.3v: track 170.9 -> 10.8 mm, vias 10 -> 0
- net /RB7: track 153.1 -> 0.00 mm, vias 5 -> 0
- net /RB6: track 141.2 -> 0.00 mm, vias 5 -> 0
- net (no net): track 130.9 -> 0.00 mm
- net /RB5: track 129.8 -> 0.00 mm, vias 5 -> 0
- net /RB1: track 120.7 -> 0.00 mm, vias 6 -> 0
- net /RD4: track 117.8 -> 0.00 mm, vias 7 -> 0
- net /MCLR: track 116.3 -> 0.00 mm, vias 4 -> 0
- net /RD6: track 113.9 -> 0.00 mm, vias 5 -> 0
- net /RB0: track 104.0 -> 0.00 mm, vias 1 -> 0
- net /RD7: track 103.2 -> 0.00 mm, vias 4 -> 0
- net /RD1: track 100.7 -> 0.00 mm, vias 9 -> 0
- net /RD3: track 100.2 -> 0.00 mm, vias 3 -> 0
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
Commit message: JaPic
Parts:
- removed G***: LOGO, FIMEE:usb_logo
- added G1: LOGO, FIMEE:github, B.Cu at (85.6, 35.1)
- C4: moved to F.Cu
- G2: footprint FIMEE:kicad_logo -> FIMEE:open_hardware
- G3: footprint FIMEE:open_hardware -> FIMEE:kicad_logo
- G4: footprint FIMEE:github -> FIMEE:abeja_sf; moved to F.Cu
- G6: footprint FIMEE:abeja_sf -> FIMEE:usb_logo
- moved H2 91.5 mm to (45.7, 95.5)
- moved J14 85.9 mm to (106.0, 30.6), turned to 0 degrees
- moved J11 77.9 mm to (93.5, 21.6), turned to 90 degrees
- moved J12 76.9 mm to (41.4, 80.5), turned to 270 degrees
- moved H4 71.2 mm to (103.6, 24.3)
- moved SW1 68.1 mm to (47.8, 21.6), turned to 0 degrees
- moved J2 66.6 mm to (106.2, 48.3)
- moved G3 60.8 mm to (99.6, 35.6), turned to 180 degrees
- moved J7 60.7 mm to (106.2, 71.4), turned to 0 degrees
- moved G4 58.0 mm to (91.9, 36.7), turned to 0 degrees
- moved H3 57.2 mm to (103.0, 95.3)
- moved C8 56.4 mm to (46.2, 30.2)
- moved INT2 55.0 mm to (97.8, 50.4)
- moved J5 54.0 mm to (58.2, 21.8), turned to 90 degrees
- moved R23 51.4 mm to (101.9, 45.2), turned to 0 degrees
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Connections:
- C4 pad 1: Net-(C3-Pad1) -> 5V
- D1 pad 2: Net-(C3-Pad1) -> 5V
- U4 pad 2: Net-(C3-Pad1) -> 5V
- U5 pad 3: Net-(C3-Pad1) -> 5V
Routing:
- net /RC5: track 111.1 -> 33.4 mm, vias 3 -> 2
- net /RC4: track 94.3 -> 31.5 mm, vias 2 -> 3
- net GND: track 87.1 -> 29.7 mm, vias 3 -> 0
- net 5V: track 0.00 -> 25.3 mm, vias 0 -> 1
- net /Vin: track 37.3 -> 25.1 mm, vias 0 -> 1
- net Net-(C3-Pad1): track 34.6 -> 43.4 mm
- net 3.3v: track 10.8 -> 6.30 mm
- net Net-(R10-Pad2): track 2.91 -> 5.45 mm
- net Net-(R1-Pad2): track 3.12 -> 5.66 mm
- net Net-(C9-Pad1): track 15.1 -> 17.4 mm
Other:
- board text added: "PGM"
- board text removed: "INT0"
- board text removed: "INT1"
- board text removed: "INT2"
