File: pic18/pic18.kicad_pcb (KiCad board)
At the start: 2 copper layers, 71.1 x 80.4 mm, 96 parts, among them J1 PORTA, J10 PORTE, J11 5v-3.3v, J12 5v-3.3v, J14 PICKIT3, J15 CONTROL, J2 PORTB, J20 LED'S, J21 BUZZER, J3 Barrel_Jack_Switch, J4 Vin, J5 TECLADO, J6 OLED, J7 PORTD, J8 HC-05, J9 PORTC, SW1 SW_Push, SW2 SW_DIP_x01, U1 PIC18F45K50, U2 3x7Segment, U3 NRF24L01_Breakout, U4 AMS1117-5.0, U5 AMS1117-3.3

Commit message: JaPic
Parts:
- moved R9 4.52 mm to (60.2, 61.2)
Connections:
- C3 pad 1: Net-(C3-Pad1) -> 5V
Routing:
- net GND: track 29.7 -> 171.4 mm, vias 0 -> 3
- net /RB1: track 0.00 -> 105.7 mm, vias 0 -> 6
- net /RB0: track 0.00 -> 104.2 mm, vias 0 -> 3
- net /RB7: track 0.00 -> 83.9 mm, vias 0 -> 1
- net /RB6: track 0.00 -> 81.1 mm, vias 0 -> 1
- net /RB5: track 0.00 -> 78.8 mm, vias 0 -> 1
- net /RB2: track 0.00 -> 74.0 mm, vias 0 -> 4
- net /RB3: track 0.00 -> 73.1 mm
- net /RB4: track 0.00 -> 72.9 mm, vias 0 -> 1
- net 5V: track 25.3 -> 70.2 mm
- net Net-(C3-Pad1): track 43.4 -> 0.00 mm
- net /RC7: track 0.00 -> 37.4 mm
- net 3.3v: track 6.30 -> 41.4 mm
- net /RA6: track 0.00 -> 32.3 mm
- net /GND1: track 0.00 -> 30.6 mm
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