File: pic18/pic18.sch (KiCad schematic (older format))
At the start: 79 parts, among them J1 PORTA, J10 PORTD, J11 PORTD1, J12 PORTC, J13 PORTC1, J14 PICKIT3, J15 CONTROL, J16 5V, J17 3.3V, J18 5V, J19 3.3V, J2 PORTB, J20 LED'S, J21 BUZZER, J22 PORTE, J23 PORTE1, J3 USB_B, J4 Barrel_Jack_Switch, J5 TECLADO, J6 LCD, J7 PORTA1, J8 HC-05, J9 PORTB1, Q1 2N3906, SW1 SW_Push, SW2 SW_DIP_x01, U1 PIC18F45K50, U3 NRF24L01_Breakout

Commit message: javimenba
Parts:
- removed J3: USB_B, Connector_USB:USB_B_OST_USB-B1HSxx_Horizontal, symbol Connector:USB_B
- removed J6: LCD, Connector_PinSocket_2.54mm:PinSocket_1x16_P2.54mm_Vertical, symbol Connector_Generic:Conn_01x16
- removed R10, R20: 220, Resistor_SMD:R_1206_3216Metric, symbol Device:R
- removed R21: 1k, Resistor_SMD:R_1206_3216Metric, symbol Device:R
- added J3: USB_B_Micro, Connector_USB:USB_Micro-B_Wuerth_629105150521, symbol Connector:USB_B_Micro
- added J6: Conn_01x04, Connector_PinSocket_2.54mm:PinSocket_1x04_P2.54mm_Vertical, symbol Connector_Generic:Conn_01x04
- 3.3v1, 5v1: symbol Regulator_Linear:L7805 -> pic18-rescue:L7805-Regulator_Linear
- BZ1: symbol Device:Buzzer -> pic18-rescue:Buzzer-Device
- C1, C2, C3, C4, C5, C6, C7, C8: symbol Device:C -> pic18-rescue:C-Device
- D1, D2: symbol Diode:1N4148 -> pic18-rescue:1N4148-Diode
- D10, D11, D12, D13, D3, D4, D5, D6, D7, D8, D9: symbol Device:LED -> pic18-rescue:LED-Device
- H1, H2, H3, H4: symbol Mechanical:MountingHole -> pic18-rescue:MountingHole-Mechanical
- J1, J10, J11, J2, J5, J7, J9: symbol Connector_Generic:Conn_01x08 -> pic18-rescue:Conn_01x08-Connector_Generic
- J12, J13, J15, J20, J21, J22, J23: symbol Connector_Generic:Conn_01x03 -> pic18-rescue:Conn_01x03-Connector_Generic
- J14: symbol Connector:Conn_01x06_Male -> pic18-rescue:Conn_01x06_Male-Connector
- J16, J17, J18, J19: symbol Connector_Generic:Conn_01x02 -> pic18-rescue:Conn_01x02-Connector_Generic
- J4: symbol Connector:Barrel_Jack_Switch -> pic18-rescue:Barrel_Jack_Switch-Connector
- J8: symbol Connector_Generic:Conn_01x06 -> pic18-rescue:Conn_01x06-Connector_Generic
- Q1: symbol Transistor_BJT:2N3906 -> pic18-rescue:2N3906-Transistor_BJT
- R1, R11, R12, R13, R14, R15, R16, R17, R18, R19, R2, R22, R3, R4, R5, R6, R7, R8, R9: symbol Device:R -> pic18-rescue:R-Device
- RV1: symbol Device:R_POT_TRIM -> pic18-rescue:R_POT_TRIM-Device
- SW1: symbol Switch:SW_Push -> pic18-rescue:SW_Push-Switch
- SW2: symbol Switch:SW_DIP_x01 -> pic18-rescue:SW_DIP_x01-Switch
- U1: symbol pic18f45k50:PIC18F45K50 -> pic18-rescue:PIC18F45K50-pic18f45k50
- U3: symbol RF:NRF24L01_Breakout -> pic18-rescue:NRF24L01_Breakout-RF
Connections:
- wire segments 283 -> 267
- no-connect marks 9 -> 6
Other:
- moved on the sheet: C8, R19

Commit message: JaPic
Parts:
- removed J3: USB_B_Micro, Connector_USB:USB_Micro-B_Wuerth_629105150521, symbol Connector:USB_B_Micro
- removed R1: 10K, Resistor_SMD:R_1206_3216Metric, symbol pic18-rescue:R-Device
- added Q2, Q3, Q4: 2N2219, Package_TO_SOT_THT:TO-92_Inline, symbol Transistor_BJT:2N2219
- added R1, R10: 5.1k, Resistor_SMD:R_1206_3216Metric, symbol Device:R
- added R20, R21, R23: 10k, Resistor_SMD:R_1206_3216Metric, symbol pic18-rescue:R-Device
- added R24, R33, R37: 10K, Resistor_SMD:R_1206_3216Metric, symbol Device:R
- added R25, R26, R27, R28, R29, R30, R31, R32: 1K, Resistor_SMD:R_1206_3216Metric, symbol Device:R
- added SW3, SW4, SW5: SW_Push, Button_Switch_SMD:SW_SPST_CK_RS282G05A3, symbol pic18-rescue:SW_Push-Switch
- added U2: 3x7Segment, Javi-7SegDisplays:3x7SEGMENT-04x08-Red, symbol 3x7Segment1:3x7Segment
- added USB1: HRO-TYPE-C-31-M-12, TypeC:HRO-TYPE-C-31-M-12-HandSoldering, symbol pic18-rescue:HRO-TYPE-C-31-M-12-Type-C
- C4: footprint Capacitor_THT:CP_Radial_D10.0mm_P2.50mm -> Capacitor_THT:CP_Radial_D5.0mm_P2.50mm
Connections:
- net GND: now also Q2.1 (E), Q3.1 (E), Q4.1 (E), R1.1, R10.1, R20.2, R21.2, R23.2, USB1.1 (GND), USB1.12 (GND), USB1.13 (SHIELD)
- net RB0: now also R20.1, R31.2, SW3.2
- net RB1: now also R21.1, R30.2, SW4.2
- net RB2: now also R23.1, R29.2, SW5.2
- net RB3: now also R28.2
- net RB4: now also R27.2
- net RB5: now also R26.2
- net RB6: now also R25.2
- net RB7: now also R32.2
- net RC4: now also USB1.5 (DN2), USB1.7 (DN1)
- net RC5: now also USB1.6 (DP1), USB1.8 (DP2)
- net RE0: now also R24.2
- net RE1: now also R33.2
- net RE2: now also R37.2
- net VDD: now also SW3.1, SW4.1, SW5.1
- net VUSB: now also USB1.11 (VBUS), USB1.2 (VBUS)
- new net: R10.2, USB1.10 (CC2)
- new net: R1.2, USB1.4 (CC1)
- new net: R25.1, U2.11 (A)
- new net: R26.1, U2.7 (B)
- new net: R27.1, U2.4 (C)
- new net: R28.1, U2.2 (D)
- new net: R29.1, U2.1 (E)
- new net: R30.1, U2.10 (F)
- new net: R32.1, U2.3 (DP)
- new net: R31.1, U2.5 (G)
- new net: Q2.2 (B), R24.1
- new net: Q3.2 (B), R33.1
- new net: Q4.2 (B), R37.1
- new net DIG1: Q2.3 (C), U2.12 (DIG1)
- new net DIG2: Q3.3 (C), U2.9 (DIG2)
- new net DIG3: Q4.3 (C), U2.8 (DIG3)
- no-connect marks 6 -> 5
Other:
- note added: "7 SEGMENTOS"
- note added: "OLED\n\n"
- note added: "RESISTENCIA\nPULL-DOWN\n"
- note removed: "LCD\n"

Commit message: JaPic
Parts:
- removed 3.3v1, 5v1: L7805, Package_TO_SOT_THT:TO-220-3_Vertical, symbol pic18-rescue:L7805-Regulator_Linear
- removed C3, C5, C7: 100nf, Capacitor_SMD:C_1206_3216Metric, symbol pic18-rescue:C-Device
- removed C4: 220uf, Capacitor_THT:CP_Radial_D5.0mm_P2.50mm, symbol pic18-rescue:C-Device
- removed C6: 0.33uf, Capacitor_THT:CP_Radial_D5.0mm_P2.50mm, symbol pic18-rescue:C-Device
- removed D1, D2: 1N4148, Diode_THT:D_DO-35_SOD27_P7.62mm_Horizontal, symbol pic18-rescue:1N4148-Diode
- removed D3: LED, LED_SMD:LED_0805_2012Metric, symbol pic18-rescue:LED-Device
- removed H1, H2, H3, H4: MountingHole, MountingHole:MountingHole_4mm_Pad_Via, symbol pic18-rescue:MountingHole-Mechanical
- removed J1: PORTA, Connector_PinSocket_2.54mm:PinSocket_1x08_P2.54mm_Vertical, symbol pic18-rescue:Conn_01x08-Connector_Generic
- removed J10: PORTD, Connector_PinSocket_2.54mm:PinSocket_1x08_P2.54mm_Vertical, symbol pic18-rescue:Conn_01x08-Connector_Generic
- removed J11: PORTD1, Connector_PinSocket_2.54mm:PinSocket_1x08_P2.54mm_Vertical, symbol pic18-rescue:Conn_01x08-Connector_Generic
- removed J12: PORTC, Connector_PinSocket_2.54mm:PinSocket_1x03_P2.54mm_Vertical, symbol pic18-rescue:Conn_01x03-Connector_Generic
- removed J13: PORTC1, Connector_PinSocket_2.54mm:PinSocket_1x03_P2.54mm_Vertical, symbol pic18-rescue:Conn_01x03-Connector_Generic
- removed J16, J18: 5V, Connector_PinSocket_2.54mm:PinSocket_1x02_P2.54mm_Vertical, symbol pic18-rescue:Conn_01x02-Connector_Generic
- removed J17, J19: 3.3V, Connector_PinSocket_2.54mm:PinSocket_1x02_P2.54mm_Vertical, symbol pic18-rescue:Conn_01x02-Connector_Generic
- removed J2: PORTB, Connector_PinSocket_2.54mm:PinSocket_1x08_P2.54mm_Vertical, symbol pic18-rescue:Conn_01x08-Connector_Generic
- removed J22: PORTE, Connector_PinSocket_2.54mm:PinSocket_1x03_P2.54mm_Vertical, symbol pic18-rescue:Conn_01x03-Connector_Generic
- removed J23: PORTE1, Connector_PinSocket_2.54mm:PinSocket_1x03_P2.54mm_Vertical, symbol pic18-rescue:Conn_01x03-Connector_Generic
- removed J4: Barrel_Jack_Switch, Connector_BarrelJack:BarrelJack_Horizontal, symbol pic18-rescue:Barrel_Jack_Switch-Connector
- removed J7: PORTA1, Connector_PinSocket_2.54mm:PinSocket_1x08_P2.54mm_Vertical, symbol pic18-rescue:Conn_01x08-Connector_Generic
- removed J9: PORTB1, Connector_PinSocket_2.54mm:PinSocket_1x08_P2.54mm_Vertical, symbol pic18-rescue:Conn_01x08-Connector_Generic
- removed Q1: 2N3906, Package_TO_SOT_THT:TO-92_Inline, symbol pic18-rescue:2N3906-Transistor_BJT
- removed R2, R3: 5.6k, Resistor_SMD:R_1206_3216Metric, symbol pic18-rescue:R-Device
- removed R4: 10k, Resistor_SMD:R_1206_3216Metric, symbol pic18-rescue:R-Device
- removed R5: 470, Resistor_SMD:R_1206_3216Metric, symbol pic18-rescue:R-Device
- added C3: 100uF, Capacitor_THT:CP_Radial_D5.0mm_P2.50mm, symbol Device:CP
- added C4, C5, C9: 0.1uF, Capacitor_SMD:C_0805_2012Metric, symbol Device:C
- added D1: LED, LED_SMD:LED_0805_2012Metric, symbol Device:LED
- added D14: 1N4007, Diode_SMD:D_1210_3225Metric_Pad1.42x2.65mm_HandSolder, symbol Diode:1N4007
- added H1: 1, MountingHole:MountingHole_4mm_Pad_Via, symbol Mechanical:MountingHole_Pad
- added H2: 2, MountingHole:MountingHole_4mm_Pad_Via, symbol Mechanical:MountingHole_Pad
- added H3: 3, MountingHole:MountingHole_4mm_Pad_Via, symbol Mechanical:MountingHole_Pad
- added H4: 4, MountingHole:MountingHole_4mm_Pad_Via, symbol Mechanical:MountingHole_Pad
- added J1: PORTA, Connector_PinSocket_2.54mm:PinSocket_2x08_P2.54mm_Vertical, symbol Connector_Generic:Conn_02x08_Odd_Even
- added J10: PORTE, Connector_PinSocket_2.54mm:PinSocket_2x03_P2.54mm_Vertical, symbol Connector_Generic:Conn_02x03_Odd_Even
- added J11, J12: 5v-3.3v, Connector_PinSocket_2.54mm:PinSocket_2x02_P2.54mm_Vertical, symbol Connector_Generic:Conn_02x02_Odd_Even
- added J2: PORTB, Connector_PinSocket_2.54mm:PinSocket_2x08_P2.54mm_Vertical, symbol Connector_Generic:Conn_02x08_Odd_Even
- added J3: Barrel_Jack_Switch, Connector_BarrelJack:BarrelJack_Wuerth_6941xx301002, symbol conectores:Barrel_Jack_Switch
- added J4: Vin, Connector_PinHeader_2.54mm:PinHeader_1x02_P2.54mm_Vertical, symbol conectores:Conn_01x02_Female
- added J7: PORTD, Connector_PinSocket_2.54mm:PinSocket_2x08_P2.54mm_Vertical, symbol Connector_Generic:Conn_02x08_Odd_Even
- added J9: PORTC, Connector_PinSocket_2.54mm:PinSocket_2x03_P2.54mm_Vertical, symbol Connector_Generic:Conn_02x03_Odd_Even
- added R2, R3, R4, R5: 4.7, Resistor_SMD:R_0805_2012Metric, symbol Device:R
- added R34: 470, Resistor_SMD:R_0805_2012Metric, symbol Device:R
- added U4: AMS1117-5.0, Package_TO_SOT_SMD:SOT-223-3_TabPin2, symbol Regulator_Linear:AMS1117-5.0
- added U5: AMS1117-3.3, Package_TO_SOT_SMD:SOT-223-3_TabPin2, symbol Regulator_Linear:AMS1117-3.3
- D10: value LED -> LED10
- D11, D5: value LED -> LED11
- D4: value LED -> LED4
- D6: value LED -> LED6
- D7: value LED -> LED7
- D8: value LED -> LED8
- D9: value LED -> LED9
- J6: value Conn_01x04 -> OLED
- R1, R10, R11, R12, R13, R14, R15, R16, R17, R18, R19, R20, R21, R22, R23, R24, R25, R26, R27, R28, R29, R30, R31, R32, R33, R37, R6, R7, R8, R9: footprint Resistor_SMD:R_1206_3216Metric -> Resistor_SMD:R_0805_2012Metric
- renumbered Q2 to DIG1, Q3 to DIG2, Q4 to DIG3, SW3 to INT0, SW4 to INT1, SW5 to INT2
Connections:
- net VUSB is gone; now on net 5V: USB1.11 (VBUS), USB1.2 (VBUS)
- net 3.3v: now also C5.1, J11.2 (Pin_2), J12.2 (Pin_2), U5.2 (VO)
- net GND: now also C3.2, C4.2, C5.2, C9.2, H1.1, H2.1, H3.1, H4.1, J11.3 (Pin_3), J11.4 (Pin_4), J12.3 (Pin_3), J12.4 (Pin_4), J3.2, J3.3, J4.2 (Pin_2), R34.2, U4.1 (GND), U5.1 (GND)
- net RA0: now also J1.1 (Pin_1), J1.2 (Pin_2)
- net RA1: now also J1.3 (Pin_3), J1.4 (Pin_4)
- net RA2: now also J1.5 (Pin_5), J1.6 (Pin_6)
- net RA3: now also J1.7 (Pin_7), J1.8 (Pin_8)
- net RA4: now also J1.10 (Pin_10), J1.9 (Pin_9)
- net RA5: now also J1.11 (Pin_11), J1.12 (Pin_12)
- net RA6: now also J1.13 (Pin_13), J1.14 (Pin_14)
- net RA7: now also J1.15 (Pin_15), J1.16 (Pin_16)
- net RB0: now also J2.1 (Pin_1), J2.2 (Pin_2); no longer R31.2
- net RB1: now also J2.3 (Pin_3), J2.4 (Pin_4); no longer R30.2
- net RB2: now also J2.5 (Pin_5), J2.6 (Pin_6); no longer R29.2
- net RB3: now also J2.7 (Pin_7), J2.8 (Pin_8); no longer R28.2
- net RB4: now also J2.10 (Pin_10), J2.9 (Pin_9); no longer R27.2
- net RB5: now also J2.11 (Pin_11), J2.12 (Pin_12); no longer R26.2
- net RB6: now also J2.13 (Pin_13), J2.14 (Pin_14); no longer R25.2
- net RB7: now also J2.15 (Pin_15), J2.16 (Pin_16); no longer R32.2
- net RC0: now also J9.1 (Pin_1), J9.2 (Pin_2)
- net RC1: now also J9.3 (Pin_3), J9.4 (Pin_4)
- net RC2: now also J9.5 (Pin_5), J9.6 (Pin_6)
- net RD0: now also R31.2, J7.1 (Pin_1), J7.2 (Pin_2)
- net RD1: now also R30.2, J7.3 (Pin_3), J7.4 (Pin_4)
- net RD2: now also R29.2, J7.5 (Pin_5), J7.6 (Pin_6)
- net RD3: now also R28.2, J7.7 (Pin_7), J7.8 (Pin_8)
- net RD4: now also R27.2, J7.10 (Pin_10), J7.9 (Pin_9)
- net RD5: now also R26.2, J7.11 (Pin_11), J7.12 (Pin_12)
- net RD6: now also R25.2, J7.13 (Pin_13), J7.14 (Pin_14)
- net RD7: now also R32.2, J7.15 (Pin_15), J7.16 (Pin_16)
- net RE0: now also J10.1 (Pin_1), J10.2 (Pin_2)
- net RE1: now also J10.3 (Pin_3), J10.4 (Pin_4)
- net RE2: now also J10.5 (Pin_5), J10.6 (Pin_6)
- net VDD: now also J11.1 (Pin_1), J12.1 (Pin_1), R2.1; no longer C1.1, U1.11 (VDD), U1.32 (VDD)
- new net: C1.1, R5.2, U1.11 (VDD)
- new net: D1.1 (K), R34.1
- new net: C3.1, C4.1, D1.2 (A), U4.2 (VO), U5.3 (VI)
- new net: C9.1, D14.1 (K), U4.3 (VI)
- new net: R2.2, R3.1
- new net: R3.2, R4.1
- new net: R4.2, R5.1
- new net Vin: D14.2 (A), J3.1, J4.1 (Pin_1)
- no-connect marks 5 -> 7
Other:
- note removed: "REGULADOR"
- moved on the sheet: BZ1, C8, D10, D11, D12, D13, D4, D5, D6, D7, D8, D9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

Commit message: JaPic
Connections:
- net 5V: now also C4.1, D1.2 (A), U4.2 (VO), U5.3 (VI)
- now unconnected: C3.1
Changed lines of the file:
@@
 	3100 6500 3400 6500
 Connection ~ 3400 6500
-Wire Wire Line
-	3400 6500 3970 6500
-Connection ~ 3970 6500
-Wire Wire Line
-	3970 6500 4620 6500
-Wire Wire Line
-	3975 5725 3975 6100
-Wire Wire Line
-	3975 6100 4450 6100
-Connection ~ 3975 6100
-Wire Wire Line
-	3975 6100 3975 6500
-Text GLabel 4450 6100 2    50   Input ~ 0
-5V
-Text Label 3975 5725 0    50   ~ 0
+Text Label 3925 5550 0    50   ~ 0
 VUSB
 $Comp
@@
 Text Label 11300 6250 0    50   ~ 0
 GND1
+Wire Wire Line
+	3925 5550 3925 5925
+Wire Wire Line
+	3925 5925 4400 5925
+Text GLabel 4400 5925 2    50   Input ~ 0
+5V
+Wire Wire Line
+	3400 6500 3975 6500
+Wire Wire Line
+	3975 6500 3975 6325
+Connection ~ 3975 6500
+Wire Wire Line
+	3975 6500 4620 6500
+Text Label 3975 6325 0    89   ~ 0
+5v
+Wire Wire Line
+	3925 5925 3725 5925
+Connection ~ 3925 5925
+Text Label 3725 5925 0    89   ~ 0
+5v
 $EndSCHEMATC

Commit message: JaPic
Connections:
- net 5V: now also C3.1
Changed lines of the file:
@@
 	1    0    0    -1
 $EndComp
-Connection ~ 4620 6500
-Wire Wire Line
-	5120 6500 4620 6500
 Wire Wire Line
 	4620 6650 4620 6500
@@
 Wire Wire Line
 	3100 6500 3400 6500
-Connection ~ 3400 6500
 Text Label 3925 5550 0    50   ~ 0
 VUSB
@@
 5V
 Wire Wire Line
-	3400 6500 3975 6500
-Wire Wire Line
 	3975 6500 3975 6325
-Connection ~ 3975 6500
-Wire Wire Line
-	3975 6500 4620 6500
 Text Label 3975 6325 0    89   ~ 0
 5v
@@
 Text Label 3725 5925 0    89   ~ 0
 5v
+Wire Wire Line
+	3975 6500 3970 6500
+Connection ~ 3400 6500
+Connection ~ 3970 6500
+Wire Wire Line
+	3970 6500 3400 6500
+Wire Wire Line
+	3975 6500 4620 6500
+Connection ~ 4620 6500
+Wire Wire Line
+	4620 6500 5120 6500
 $EndSCHEMATC
